Commit message: added small car parameters

File: sample_vehicle_description/urdf/vehicle.xacro (robot description, xacro)
@@ -6,5 +6,5 @@
   <link name="base_link">
     <visual>
-      <origin xyz="${vehicle_info['/**']['ros__parameters']['wheel_base']/2.0} 0 0" rpy="${pi/2.0} 0 ${pi}"/>
+      <origin xyz="2.4 -3.1 0" rpy="0 0 ${pi/2.0}"/>
       <geometry>
         <mesh filename="package://sample_vehicle_description/mesh/lexus.dae" scale="1 1 1"/>
